Commit message: First commit to master

File: panasonic_vr006l/panasonic_vr006l_support/urdf/panasonic.urdf (robot description, URDF)
Before this commit: robot panasonic, 7 links, 6 joints
Links:
- link link3: geometry visual mesh filename=package://panasonic_vr006l_support/meshes/cad/elbow_new.stl scale=.01 .01 .01
- link link4: geometry visual mesh filename=package://panasonic_vr006l_support/meshes/cad/forearm_new.s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 scale=.01 .01 .01
Joints:
- joint joint_link4_link5: origin xyz=0 -0.25 0.001 rpy=0 0 0 -> xyz=0 -0.25 0.001 rpy=1.57 0 0
